Commit message: Add files via upload

File: ros2_ws/src/last_description/urdf/last.xacro (robot description, xacro)
@@ -331,4 +331,9 @@
       <state_interface name="position"/>
     </joint>
+    <joint name="zed_camera_joint" type="fixed">
+      <parent link="base_link"/> <!-- ya da kameranın bağlı olacağı link -->
+      <child link="zed_camera_link"/>
+      <origin xyz="1.05 0.35 0.34" rpy="0 0 0"/> <!-- Burayı istediğin pozisyona göre ayarlayabilirsin -->
+    </joint>
   </ros2_control>
 </robot>

File: ros2_ws/src/last_description/urdf/lidar.xacro (robot description, xacro)
@@ -4,23 +4,21 @@
         <parent link="base_link"/>
         <child link="laser_frame"/>
-        <origin xyz="0.1 0 0.175" rpy="0 0 0"/>
+        <origin xyz="0.95 0.41 0.45" rpy="0 0 0"/>
     </joint>
     <link name="laser_frame">
         <visual>
-            <origin xyz="-1.032099 0.3925 0.402901" rpy="0 0 0"/>
             <geometry>
-                <mesh filename="file://$(find last_description)/meshes/right_fornt_wheel_v1_1.stl" scale="0.001 0.001 0.001"/>
+                <cylinder radius="0.04" length="0.06"/>
             </geometry>
             <material name="silver"/>
         </visual>
         <collision>
-            <origin xyz="-1.032099 0.3925 0.402901" rpy="0 0 0"/>
             <geometry>
-                <mesh filename="file://$(find last_description)/meshes/right_fornt_wheel_v1_1.stl" scale="0.001 0.001 0.001"/>
+                <cylinder radius="0.04" length="0.06"/>
             </geometry>
         </collision>
     </link>
     <gazebo reference="laser_frame">
-        <material>Gazebo/silver</material>
+        <material>Gazebo/Red</material>
         <sensor name="laser" type="ray">
             <pose> 0 0 0 0 0 0 </pose>
